File: hw/uv39_res/uv39_res.kicad_pcb (KiCad board)
At the start: 2 copper layers, 48.9 x 27.4 mm, 18 parts, among them J1 ATF13-3P-BM03, J2 ATF13-2P-BM03, J3 90HBW06PT

Commit message: 1.1.0 silkscreen fixes
Other:
- board text added: "0"
- board text added: "1.1.0"

Commit message: DT063S pin out fixed
Routing:
- net GND: track 50.8 -> 0.00 mm
- net Net-(J1-2): track 52.6 -> 64.3 mm
- net Net-(J1-1): track 35.6 -> 30.8 mm
Other:
- board text added: "1.2.0"
- board text removed: "1.1.0"
Changed lines of the file:
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@@
 		)
 		(pad "B" thru_hole circle
-			(at 0 0 90)
+			(at 4.3 0 90)
 			(size 2.4 2.4)
 			(drill 1.7)
@@
 		)
 		(pad "C" thru_hole circle
-			(at 4.3 0 90)
+			(at 0 0 90)
 			(size 2.4 2.4)
 			(drill 1.7)
@@
 		)
 	)
-	(gr_text "1.1.0"
+	(gr_text "1.2.0"
 		(at 118.398335 111.876714 0)
 		(layer "F.SilkS")
@@
 	)
 	(segment
-		(start 103.8 101.1)
-		(end 106 103.3)
+		(start 110.45 99.25)
+		(end 110.45 96.8)
 		(width 0.25)
 		(layer "F.Cu")
@@
 	)
 	(segment
-		(start 104.8 96.8)
-		(end 103.8 97.8)
-		(width 0.25)
-		(layer "F.Cu")
-		(net 1)
-	)
-	(segment
-		(start 103.8 97.8)
-		(end 103.8 101.1)
-		(width 0.25)
-		(layer "F.Cu")
-		(net 1)
-	)
-	(segment
 		(start 127.1 90.35)
 		(end 124.3229 90.35)
@@
 	)
 	(segment
-		(start 111 96.8)
-		(end 104.8 96.8)
+		(start 106 103.7)
+		(end 110.45 99.25)
 		(width 0.25)
 		(layer "F.Cu")
@@
 	)
 	(segment
+		(start 111 96.8)
+		(end 110.45 96.8)
+		(width 0.25)
+		(layer "F.Cu")
+		(net 1)
+	)
+	(segment
 		(start 128 92)
 		(end 128 91.25)
@@
 	)
 	(segment
+		(start 103 103.35)
+		(end 103 96.6)
+		(width 0.25)
+		(layer "F.Cu")
+		(net 2)
+	)
+	(segment
 		(start 144.4 98.6)
 		(end 141.2 98.6)
@@
 	)
 	(segment
-		(start 109 101.8)
-		(end 111.345 104.145)
-		(width 0.25)
-		(layer "F.Cu")
-		(net 2)
-	)
-	(segment
-		(start 107.989874 99)
-		(end 109 100.010126)
+		(start 103 96.6)
+		(end 104.5 95.1)
 		(width 0.25)
 		(layer "F.Cu")
@@
 	)
 	(segment
-		(start 111.345 104.145)
-		(end 116.1962 104.145)
-		(width 0.25)
-		(layer "F.Cu")
-		(net 2)
-	)
-	(segment
-		(start 109 100.010126)
-		(end 109 101.8)
+		(start 112.65 104.145)
+		(end 111.195 105.6)
+		(width 0.25)
+		(layer "F.Cu")
+		(net 2)
+	)
+	(segment
+		(start 105.25 105.6)
+		(end 103 103.35)
 		(width 0.25)
 		(layer "F.Cu")
@@
 	)
 	(segment
+		(start 111.195 105.6)
+		(end 105.25 105.6)
+		(width 0.25)
+		(layer "F.Cu")
+		(net 2)
+	)
+	(segment
 		(start 116.1962 104.145)
 		(end 116.1962 102)
@@
 	)
 	(segment
-		(start 106 99)
-		(end 107.989874 99)
+		(start 104.5 95.1)
+		(end 106 95.1)
+		(width 0.25)
+		(layer "F.Cu")
+		(net 2)
+	)
+	(segment
+		(start 116.1962 104.145)
+		(end 112.65 104.145)
 		(width 0.25)
 		(layer "F.Cu")
@@
 	)
 	(segment
-		(start 140.09735 87.2)
-		(end 147.2 94.30265)
-		(width 0.25)
-		(layer "F.Cu")
-		(net 3)
-	)
-	(segment
-		(start 111.510126 87.2)
-		(end 140.09735 87.2)
-		(width 0.25)
-		(layer "F.Cu")
-		(net 3)
-	)
-	(segment
-		(start 147.2 94.30265)
-		(end 147.2 96.7)
-		(width 0.25)
-		(layer "F.Cu")
-		(net 3)
-	)
-	(segment
-		(start 106 94.7)
-		(end 106 92.710126)
-		(width 0.25)
-		(layer "F.Cu")
-		(net 3)
-	)
-	(segment
-		(start 106 92.710126)
-		(end 111.510126 87.2)
-		(width 0.25)
-		(layer "F.Cu")
-		(net 3)
-	)
-	(segment
